Commit message: test

File: km_robot.urdf (robot description, URDF)
Before this commit: robot quadruped_robot, 22 links, 21 joints
Links:
- link FL_calf: mass 0.0021743238101132596 -> 2.3268485144669113; geometry visual cylinder length=0.2675220349037209 radius=0.0429619227247509
- link FL_foot: mass 0.00018492113189266972 -> 0.15267296851711973; geometry collision sphere radius=0.02896414817135573; visual sphere radius=0.02896414817135573
- link FL_hip: mass 0.00022932322639885932 -> 0.4451106953851888; geometry visual sphere radius=0.04137735453050819
- link FL_knee: mass 0.0004655652060141283 -> 0.4982312882835031; geometry visual sphere radius=0.0429619227247509
- link FL_thigh: mass 0.0035319234883072845 -> 2.6304486108259537; geometry visual cylinder length=0.3260342677986043 radius=0.04137735453050819
- link FR_calf: mass 0.0021896533585434724 -> 2.3268485144669113; geometry visual cylinder length=0.2675220349037209 radius=0.0429619227247509
- link FR_foot: mass 0.0002211679474225979 -> 0.15267296851711973; geometry collision sphere radius=0.02896414817135573; visual sphere radius=0.02896414817135573
- link FR_hip: mass 0.0007133946346302859 -> 0.4451106953851888; geometry visual sphere radius=0.04137735453050819
- link FR_knee: mass 0.0005897571161158912 -> 0.4982312882835031; geometry visual sphere radius=0.0429619227247509
- link FR_thigh: mass 0.002595583183064086 -> 2.6304486108259537; geometry visual cylinder length=0.3260342677986043 radius=0.04137735453050819
- link RL_calf: mass 0.0012361981975151917 -> 2.3268485144669113; geometry visual cylinder length=0.2675220349037209 radius=0.0429619227247509
- link RL_foot: mass 0.0001796348284367131 -> 0.15267296851711973; geometry collision sphere radius=0.02896414817135573; visual sphere radius=0.02896414817135573
- link RL_hip: mass 0.0002645088064979321 -> 0.4451106953851888; geometry visual sphere radius=0.04137735453050819
- link RL_knee: mass 0.0007413487391799301 -> 0.4982312882835031; geometry visual sphere radius=0.0429619227247509
- link RL_thigh: mass 0.0039907554860377815 -> 2.6304486108259537; geometry visual cylinder length=0.3260342677986043 radius=0.04137735453050819
- link RR_calf: mass 0.002988473888183745 -> 2.3268485144669113; geometry visual cylinder length=0.2675220349037209 radius=0.0429619227247509
- link RR_foot: mass 0.00010220979717657491 -> 0.15267296851711973; geometry collision sphere radius=0.02896414817135573; visual sphere radius=0.02896414817135573
- link RR_hip: mass 0.0006461741726299969 -> 0.4451106953851888; geometry visual sphere radius=0.04137735453050819
- link RR_knee: mass 0.0006060964622261971 -> 0.4982312882835031; geometry visual sphere radius=0.0429619227247509
- link RR_thigh: mass 0.001527485349278443 -> 2.6304486108259537; geometry visual cylinder length=0.3260342677986043 radius=0.04137735453050819
- link base: mass 7.203394176650595e-07 -> None; geometry visual box size=0.01 0.01 0.01
- link trunk: mass 0.014493089404382023 -> 29.808714923389527; geometry collision box size=0.6861772090809941 0.3034325696406455 0.0954450721288132; visual box size=0.6861772090809941 0.3034325696406455 0.0954450721288132
Joints:
- joint FL_foot_joint: origin xyz=0 0 -0.28255693038374063 rpy=0 0 0 -> xyz=0 0 -0.2675220349037209 rpy=0 0 0
- joint FL_hip_joint: origin xyz=0.20087554431490998 0.17436409388922194 -0.03704724621880318 rpy=0 0 0 -> xyz=0.34308860454049706 0.15171628482032276 -0.038178028851525284 rpy=0 0 0
- joint FL_knee_joint: origin xyz=0 0 -0.33117571690571346 rpy=0 0 0 -> xyz=0 0 -0.3260342677986043 rpy=0 0 0
- joint FR_foot_joint: origin xyz=0 0 -0.28255693038374063 rpy=0 0 0 -> xyz=0 0 -0.2675220349037209 rpy=0 0 0
- joint FR_hip_joint: origin xyz=0.20087554431490998 -0.17436409388922194 -0.03704724621880318 rpy=0 0 0 -> xyz=0.34308860454049706 -0.15171628482032276 -0.038178028851525284 rpy=0 0 0
- joint FR_knee_joint: origin xyz=0 0 -0.33117571690571346 rpy=0 0 0 -> xyz=0 0 -0.3260342677986043 rpy=0 0 0
- joint RL_foot_joint: origin xyz=0 0 -0.28255693038374063 rpy=0 0 0 -> xyz=0 0 -0.2675220349037209 rpy=0 0 0
- joint RL_hip_joint: origin xyz=-0.20087554431490998 0.17436409388922194 -0.03704724621880318 rpy=0 0 0 -> xyz=-0.34308860454049706 0.15171628482032276 -0.038178028851525284 rpy=0 0 0
- joint RL_knee_joint: origin xyz=0 0 -0.33117571690571346 rpy=0 0 0 -> xyz=0 0 -0.3260342677986043 rpy=0 0 0
- joint RR_foot_joint: origin xyz=0 0 -0.28255693038374063 rpy=0 0 0 -> xyz=0 0 -0.2675220349037209 rpy=0 0 0
- joint RR_hip_joint: origin xyz=-0.20087554431490998 -0.17436409388922194 -0.03704724621880318 rpy=0 0 0 -> xyz=-0.34308860454049706 -0.15171628482032276 -0.038178028851525284 rpy=0 0 0
- joint RR_knee_joint: origin xyz=0 0 -0.33117571690571346 rpy=0 0 0 -> xyz=0 0 -0.3260342677986043 rpy=0 0 0
